Commit message: second commit

File: my_robot/urdf/my_robot.xacro (robot description, xacro)
@@ -49,17 +49,29 @@
     </inertial>
     <collision name='collision'>
-      <origin xyz="0 0 0" rpy=" 0 0 0"/>
+      <origin xyz="-0.1 0 0" rpy=" 0 0 0"/>
       <geometry>
-        <box size=".4 .2 .1"/>
+        <box size=".6 .2 .1"/>
       </geometry>
     </collision>
     <visual name='chassis_visual'>
-      <origin xyz="0 0 0" rpy=" 0 0 0"/>
+      <origin xyz="-0.1 0 0" rpy=" 0 0 0"/>
       <geometry>
-        <box size=".4 .2 .1"/>
+        <box size=".6 .2 .1"/>
+      </geometry>
+    </visual>
+    <collision name='room_collision'>
+      <origin xyz="-0.2 0 0.15" rpy=" 0 0 0"/>
+      <geometry>
+        <box size=".2 .2 .2"/>
+      </geometry>
+    </collision>
+    <visual name='room_visual'>
+      <origin xyz="-0.2 0 0.15" rpy=" 0 0 0"/>
+      <geometry>
+        <box size=".2 .2 .2"/>
       </geometry>
     </visual>
     <collision name='back_caster_collision'>
-      <origin xyz="-0.15 0 -0.05" rpy=" 0 0 0"/>
+      <origin xyz="-0.35 0 -0.05" rpy=" 0 0 0"/>
       <geometry>
         <sphere radius="0.0499"/>
@@ -67,5 +79,5 @@
     </collision>
     <visual name='back_caster_visual'>
-      <origin xyz="-0.15 0 -0.05" rpy=" 0 0 0"/>
+      <origin xyz="-0.35 0 -0.05" rpy=" 0 0 0"/>
       <geometry>
         <sphere radius="0.05"/>

Commit message: first commit

File: my_robot/urdf/my_robot.xacro (robot description, xacro)
@@ -32,4 +32,9 @@
     <limit effort="10000" velocity="1000"/>
     <dynamics damping="1.0" friction="1.0"/>
+  </joint>
+  <joint name="camera_optical_joint" type="fixed">
+    <origin xyz="0 0 0" rpy="-1.5707 0 -1.5707"/>
+    <parent link="camera"/>
+    <child link="camera_link_optical"/>
   </joint>
   <joint type="fixed" name="hokuyo_joint">
@@ -154,4 +159,6 @@
     </visual>
   </link>
+  <link name="camera_link_optical">
+  </link>
   <link name="hokuyo">
     <inertial>
